Commit message: fixed imu data, fixed odometry data, fixed transformations, use services instead of topics,

File: sphero_description/urdf/sphero.urdf (robot description, URDF)
Before this commit: robot sphero, 1 links, 0 joints
Links:
- added link base_footprint; collision box size=0.001 0.001 0.001; visual box size=0.001 0.001 0.001
- link base_link: mass 0.5 -> None; geometry collision sphere radius=0.0381; visual mesh filename=package://sphero_description/meshes/Sphero_Textured.dae
Joints:
- added joint base_footprint_joint: type continuous, parent base_footprint, child base_link, origin xyz=0 0 0.038 rpy=0 0 0
